File: PCB/HapticFeebackBoard/Haptic Feeback board.kicad_sch (KiCad schematic)
At the start: 3 parts, among them J1 Conn_01x02, J2 Conn_01x04, Q1 2N7002E

Commit message: Support on haptic feedback board
Added schematic details, imported PCBWay DRC
Other:
- company: (none) -> Running Cadence Measurement Belt
- title: (none) -> Haptic Feedback Board
