File: PCB/InertialMeasurementUnitBoard/InertialMeasurementUnitBoard.kicad_sch (KiCad schematic)
At the start: 16 parts, among them J1 1769, J2 2005280060, U1 CD74HC4050PWR, X2 SC32S-7PF20PPM

Commit message: Recovery attempt 2
Parts:
- added GND1, VDD1: TestPoint, TestPoint:TestPoint_THTPad_D2.0mm_Drill1.0mm, symbol Connector:TestPoint
- added H1, H2, H3, H4: MountingHole, MountingHole:MountingHole_3.2mm_M3, symbol Mechanical:MountingHole
Connections:
- net +3.3V: now also VDD1.1
- net GND: now also GND1.1
