File: PCB/MicrocontrollerUnitBoard/MicrocontrollerUnitBoard.kicad_sch (KiCad schematic)
At the start: 1 part, among them U1 ESP32-S3-WROOM-1

Commit message: Recovery attempt 2
Parts:
- removed U1: ESP32-S3-WROOM-1, RF_Module:ESP32-S3-WROOM-1, symbol RF_Module:ESP32-S3-WROOM-1
- added C1, C2: 0.1uF, symbol Device:C_Small
- added J1, J2: 1769, 1769, symbol Adafruit Accessories JST-PH 2-pin SMT Right Angle Connect:1769
- added J3: 2005280060, CON_2005280060_MOL, symbol WM24188TR-ND:2005280060
- added J4: 10118192-0001LF, 10118192-0001LF:AMPHENOL_10118192-0001LF, symbol AMPHENOL_10118192-0001LF:10118192-0001LF
- added R1, R2: 5.1k, symbol Device:R_Small
- added SW1, SW2: PTS526 SM15 SMTR2 LFS, SON4_PTS526 SM15 SMTR2 LFS_CNK, symbol PTS526 SM15 SMTR2 LFS:PTS526_SM15_SMTR2_LFS
- added TP1, TP10, TP11, TP12, TP2, TP3, TP4, TP5, TP6, TP7, TP8, TP9: TestPoint, symbol Connector:TestPoint
Connections:
- new net: C1.2, R1.2, SW1.3, TP11.1
- new net: C2.2, R2.2, SW2.3, TP12.1
- new net: J4.3 (D+), TP2.1
- new net: J4.2 (D-), TP1.1
- new net +3.3V: J1.1, J2.1, R1.1, R2.1, TP10.1
- new net CS_N: J3.4, TP5.1
- new net GND: C1.1, C2.1, J1.2, J2.2, J4.5 (GND), SW1.2, SW2.2, TP9.1
- new net INT_N: J3.5, TP4.1
- new net MISO: J3.2, TP7.1
- new net MOSI: J3.1, TP8.1
- new net RST_N: J3.6, TP3.1
- new net SCLK: J3.3, TP6.1
- no-connect marks 1 -> 0
