File: PCB/MicrocontrollerUnitBoard/MicrocontrollerUnitBoard.kicad_pcb (KiCad board)
At the start: 2 copper layers, 55.8 x 39.7 mm, 31 parts, among them J1 1769, J2 1769, J3 2005280060, J4 10118192-0001LF, SW1 PTS526 SM15 SMTR2 LFS, SW2 PTS526 SM15 SMTR2 LFS

Commit message: Finish MCU Test board
Parts:
- added 3.3V2: TestPoint, TestPoint:TestPoint_THTPad_D2.0mm_Drill1.0mm, F.Cu at (124.5, 115.1)
- added 3.3V3: TestPoint, TestPoint:TestPoint_THTPad_D2.0mm_Drill1.0mm, F.Cu at (127.9, 115.1)
- added 3.3V4: TestPoint, TestPoint:TestPoint_THTPad_D2.0mm_Drill1.0mm, F.Cu at (131.3, 115.1)
- added GND2: TestPoint, TestPoint:TestPoint_THTPad_D2.0mm_Drill1.0mm, F.Cu at (114.6, 85.0)
- added GND3: TestPoint, TestPoint:TestPoint_THTPad_D2.0mm_Drill1.0mm, F.Cu at (117.9, 85.0)
- added GND4: TestPoint, TestPoint:TestPoint_THTPad_D2.0mm_Drill1.0mm, F.Cu at (121.2, 85.0)
- added GND5: TestPoint, TestPoint:TestPoint_THTPad_D2.0mm_Drill1.0mm, F.Cu at (124.5, 85.0)
Routing:
- net +3.3V: track 74.9 -> 82.9 mm
